Commit message: Fixed merge problem in controller launch file, fixed joint in urdf

File: ros_ws/src/Simulation/robot_description_old/urdf/robot.urdf (robot description, URDF)
Before this commit: robot robot_description, 4 links, 3 joints
Joints:
- joint dummy_joint: type continuous -> fixed

Commit message: Turned off base collisions

File: ros_ws/src/Simulation/robot_description_old/urdf/robot.urdf (robot description, URDF)
Before this commit: robot robot_description, 4 links, 3 joints
Links:
- link base_link: geometry visual mesh filename=package://robot_description/meshes/base_link.STL
