Commit message: Half-working issimulation, controllers and encoders in place

File: ros_ws/src/Simulation/robot_description/urdf/robot.urdf (robot description, URDF)
Before this commit: robot robot_description, 4 links, 3 joints
Links:
- removed link left_wheel
- removed link right_wheel
- removed link stationary_shaft
- added link wheelL, mass 0.53129; collision mesh filename=package://robot_description/meshes/wheelL.STL; visual mesh filename=package://robot_description/meshes/wheelL.STL
- added link wheelR, mass 0.53129; collision mesh filename=package://robot_description/meshes/wheelR.STL; visual mesh filename=package://robot_description/meshes/wheelR.STL
- link base_link: mass 6.7886 -> 9.2197
Joints:
- removed joint left wheel
- removed joint right_wheel
- removed joint stationary_shaft
- added joint wheelL: type continuous, parent base_link, child wheelL, origin xyz=0.148252974079396 -0.0058042589636423 -0.433884033953984 rpy=1.5707963267949 -0.169516066406974 -1.5707963267949, axis 0 0 1
- added joint wheelR: type continuous, parent base_link, child wheelR, origin xyz=-0.207347025920604 -0.0058042589636423 -0.433884033953984 rpy=1.5707963267949 -0.169516066406974 -1.5707963267949, axis 0 0 1

Commit message: Update UI with robot model

File: ros_ws/src/Simulation/robot_description/urdf/robot.urdf (robot description, URDF)
Before this commit: robot robot_description, 3 links, 2 joints
Links:
- added link dummy_link
Joints:
- added joint dummy_joint: type continuous, parent dummy_link, child base_link, origin xyz=0 0 0 rpy=0 0 0, axis 0 0 1

Commit message: Fixed slow simulation problem! Problem was mesh collision with body, but they can be turned off by commenting out body collisions

File: ros_ws/src/Simulation/robot_description/urdf/robot.urdf (robot description, URDF)
Before this commit: robot robot_description, 4 links, 3 joints
Links:
- link base_link: geometry visual mesh filename=package://robot_description/meshes/base_link.STL
Joints:
- joint dummy_joint: type continuous -> fixed

Commit message: Using spliced together urdf

File: ros_ws/src/Simulation/robot_description/urdf/robot.urdf (robot description, URDF)
Before this commit: robot robot_description, 4 links, 3 joints
Links:
- link base_link: geometry collision mesh filename=package://robot_description/meshes/base_link.STL; visual mesh filename=package://robot_description/meshes/base_link.STL
Joints:
- joint dummy_joint: type fixed -> continuous

Commit message: Sim finally loading!

File: ros_ws/src/Simulation/robot_description/urdf/robot.urdf (robot description, URDF)
Before this commit: robot robot_description, 6 links, 5 joints
Links:
- link base_link: geometry visual mesh filename=package://robot_description/meshes/base_link.STL
- link camera: mass 0.0447522009688967 -> 0.044752
- link wheel_l: mass 0.601468487385641 -> 0.60147
- link wheel_r: mass 0.60146848738564 -> 0.60147

Commit message: Waiting on dead reckoning state estimator

File: ros_ws/src/Simulation/robot_description/urdf/robot.urdf (robot description, URDF)
Before this commit: robot robot_description, 6 links, 5 joints
Links:
- link base_link: geometry collision mesh filename=package://robot_description/meshes/base_link.STL; visual mesh filename=package://robot_description/meshes/base_link.STL
